File: power.sch (KiCad schematic (older format))
At the start: 31 parts, among them J1 Conn_SWD, M1 Vibrator, Q1 NTR5103N, SW1 Btn_Up, SW2 Btn_Down, SW3 Btn_Select, SW4 Btn_Back, U1 ATSAMD21J18A-MU

Commit message: Finish up the schematic
Parts:
- removed C1, C3, C4, C5: 0.1uF, Capacitor_SMD:C_0603_1608Metric, symbol Device:C_Small
- removed C2: 4.7uF, Capacitor_SMD:C_0603_1608Metric, symbol Device:C_Small
- removed C6: 1uF, Capacitor_SMD:C_0603_1608Metric, symbol Device:C_Small
- removed D1: LED_TopLeft, LED_SMD_Extra:LED_RGBA_0606, symbol Device_Extra:LED_RGBA
- removed D2: LED_TopRight, LED_SMD_Extra:LED_RGBA_0606, symbol Device_Extra:LED_RGBA
- removed D3: LED_BottomLeft, LED_SMD_Extra:LED_RGBA_0606, symbol Device_Extra:LED_RGBA
- removed D4: LED_BottomRight, LED_SMD_Extra:LED_RGBA_0606, symbol Device_Extra:LED_RGBA
- removed J1: Conn_SWD, Connector_JST:JST_SH_SM04B-SRSS-TB_1x04-1MP_P1.00mm_Horizontal, symbol Connector_Generic:Conn_01x04
- removed M1: Vibrator, Buzzer_Beeper_Extra:C1026B, symbol Motor:Motor_DC
- removed Q1: NTR5103N, Package_TO_SOT_SMD:SOT-23, symbol Transistor_FET:BSS138
- removed R1: 1K, Resistor_SMD:R_0603_1608Metric, symbol Device:R_Small
- removed R10, R11, R12, R13, R2, R3, R4, R5, R6, R7, R8, R9: 360R, Resistor_SMD:R_0603_1608Metric, symbol Device:R_Small
- removed SW1: Btn_Up, Button_Switch_SMD_Extra:KLS7-TS2402, symbol Switch:SW_Push
- removed SW2: Btn_Down, Button_Switch_SMD_Extra:KLS7-TS2402, symbol Switch:SW_Push
- removed SW3: Btn_Select, Button_Switch_SMD_Extra:KLS7-TS2402, symbol Switch:SW_Push
- removed SW4: Btn_Back, Button_Switch_SMD_Extra:KLS7-TS2402, symbol Switch:SW_Push
- removed U1: ATSAMD21J18A-MU, Package_DFN_QFN:QFN-64-1EP_9x9mm_P0.5mm_EP4.7x4.7mm, symbol MCU_Microchip_SAMD:ATSAMD21J18A-MU
- added BT1: CR2032, Battery_Extra:BAT-HLD-001, symbol Device:Battery_Cell
- added C7, C8: 1uF, Capacitor_SMD:C_0603_1608Metric, symbol Device:C_Small
- added D5, D6: S1JHE, Diode_SMD:D_SOD-323F, symbol Device:D_Small
- added J2: USB_B_Micro, Connector_USB:USB_Micro-B_Molex-105017-0001, symbol Connector:USB_B_Micro
- added U2: MCP1700-3302E, Package_TO_SOT_SMD:SOT-23, symbol Regulator_Linear:MCP1700-3302E_SOT23
Connections:
- net labels added: +BATT, VBUS
- net labels removed: +1V2, ACCEL_INT, ACCEL_SCL, ACCEL_SDA, BTN_BACK, BTN_DOWN, BTN_SELECT, BTN_UP, FLASH_CS, FLASH_SCK, FLASH_SI, FLASH_SO, LCD_CS, LCD_DC, LCD_DIN, LCD_RESET, LCD_SCK, LED1_B, LED1_G, LED1_R, LED2_B, LED2_G, LED2_R, LED3_B, LED3_G, LED3_R, LED4_B, LED4_G, LED4_R, MIC_CLK, MIC_DATA, RFM_CS, RFM_MISO, RFM_MOSI, RFM_RESET, RFM_SCK, SPEAKER, SPEAKER_SD, SWDCLK, SWDIO, VIBRATOR
- wire segments 154 -> 25
Other:
- note added: "Out: 250mA\nDropout: 178mV"
- note removed: "I2SD1"
- note removed: "I2SSCK"
- note removed: "SERCOM0 - Display\nSERCOM1 - Accelerometer\nSERCOM3 - Flash\nSERCOM4 - RFM"
- note removed: "SERCOM0.0"
- note removed: "SERCOM0.1"
- note removed: "SERCOM1.0"
- note removed: "SERCOM1.1"
- note removed: "SERCOM3.0"
- note removed: "SERCOM3.2\n"
- note removed: "SERCOM3.3"
- note removed: "SERCOM4.0\n"
- note removed: "SERCOM4.1"
- note removed: "SERCOM4.2"
- note removed: "TCC"
- note removed: "VOUT0"
