File: xilwatch2.kicad_pcb (KiCad board)
At the start: 2 copper layers, 35.8 x 50 mm, 63 parts, among them J1 USB_B_Micro, J2 Conn_SWD, M1 Vibrator, Q1 Si1308, Q2 NTR5103N, SW1 Btn_Up, SW2 Btn_Down, SW3 Btn_Select, SW4 Btn_Back, U1 MCP1700-3302E, U2 Holyiot_18010, U3 26VF0168IS2AE, U4 PAM8301, U5 LIS3DH

Commit message: WIP
Parts:
- removed J2: Conn_SWD, Connector_JST:JST_SH_SM04B-SRSS-TB_1x04-1MP_P1.00mm_Horizontal
- added REF**: TestPoint_Pad_D1.0mm, TestPoint:TestPoint_Pad_D1.0mm, F.Cu at (164.0, 88.8)
- added TP1: TP_GND, TestPoint:TestPoint_Pad_D1.0mm, F.Cu at (130.9, 96.4)
- added TP2: TP_VDD, TestPoint:TestPoint_Pad_D1.0mm, F.Cu at (131.1, 99.1)
- added TP3: TP_SWDCLK, TestPoint:TestPoint_Pad_D1.0mm, F.Cu at (153.8, 79.2)
- added TP4: TP_SWDIO, TestPoint:TestPoint_Pad_D1.0mm, F.Cu at (155.8, 79.2)
- added U6: GDEW0154T8, Connector_GoodDisplay:GoodDisplay_24P-0.5SH_1x24-Horizontal, B.Cu at (164.2, 96.0)
- BT1, C1, C10, C11, C12, C13, C14, C15, C16, C17, C18, C2, C3, C7, C8, C9, D1, D2, D3, D4, D5, J1, L1, M1, Q1, Q2, R3, R4, SW1, SW2, SW3, SW4, U1: moved to B.Cu
- LS1: value Speaker -> CMT-5023S-SMT; footprint Symbol:CE-Logo_8.5x6mm_SilkScreen -> Buzzer_Beeper_Extra:CMT-5023S
- R1, R2: value 360R -> 22R
- U3: value 26VF0168IS2AE -> IS25LP128F
- moved R3 77.8 mm to (81.6, 80.2)
- moved D5 77.8 mm to (84.3, 77.3)
- moved C3 77.4 mm to (90.2, 77.2)
- moved Q1 71.5 mm to (81.3, 84.7)
- moved C7 71.0 mm to (96.7, 86.3)
- moved R4 64.1 mm to (89.0, 79.6)
- moved L1 62.2 mm to (88.8, 84.4)
- moved C14 55.2 mm to (110.6, 73.3)
- moved R1 54.4 mm to (164.6, 79.9), turned to 270 degrees
- moved C9 54.4 mm to (110.7, 67.5)
- moved C12 53.1 mm to (110.7, 70.8)
- moved C11 51.1 mm to (110.8, 69.1)
- moved C13 50.2 mm to (115.4, 67.0)
- moved C17 50.2 mm to (113.0, 64.7)
- moved C16 47.5 mm to (117.2, 64.8)
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Connections:
- U3 pad 1: /QSPI_IO3 -> /QSPI_CS
- U3 pad 2: /QSPI_IO0 -> /QSPI_IO1
- U3 pad 3: /QSPI_CS -> /QSPI_IO2
- U3 pad 5: /QSPI_IO1 -> /QSPI_IO0
- U3 pad 6: /QSPI_IO2 -> /QSPI_CLK
- U3 pad 7: /QSPI_CLK -> /QSPI_IO3
- U3 pad 9: (no net) -> GND
Other:
- board size 35.8 x 50 mm -> 37.8 x 50 mm
- board text added: "1.2mm PCB!"
